Commit message: Update limo training

File: limo_bringup/description/urdf/dabai.xacro (robot description, xacro)
@@ -1,5 +1,5 @@
 <?xml version="1.0"?>
 <robot name="dabai" xmlns:xacro="http://wiki.ros.org/xacro">
-    <xacro:macro name="dabai" params="object_name:='dabai' topic='dabai' image_link='dabai_image_link' point_link='dabai_point_link' parent_link:='link' xyz:='0 0 0' rpy:='0 0 0'">
+    <xacro:macro name="dabai" params="object_name:='dabai' topic='dabai' camera_link='camera_link'  image_link='image_link' point_link='point_link' parent_link:='link' xyz:='0 0 0' rpy:='0 0 0'">
         <xacro:property
             name="mass"
@@ -18,5 +18,5 @@
             value="3.1415926536"/>
         <link
-            name="${image_link}">
+            name="${camera_link}">
             <inertial>
                 <origin
@@ -60,7 +60,9 @@
         </link>
         <link
+            name="${image_link}"/>
+        <link
             name="${point_link}"/>
         <joint
-            name="${object_name}_image_joint"
+            name="${object_name}_camera_joint"
             type="fixed">
             <origin
@@ -70,4 +72,15 @@
                 link="${parent_link}"/>
             <child
+                link="${camera_link}"/>
+        </joint>
+        <joint
+            name="${object_name}_image_joint"
+            type="fixed">
+            <origin
+                xyz="0 0.01 0"
+                rpy="0 0 0"/>
+            <parent
+                link="${camera_link}"/>
+            <child
                 link="${image_link}"/>
         </joint>
@@ -76,18 +89,36 @@
             type="fixed">
             <origin
-                xyz="0 0 0"
-                rpy="${-90*M_PI/180} ${0*M_PI/180} ${-90*M_PI/180}"/>
+                xyz="0 0.0 0"
+                rpy="0 0 0"/>
+                <!-- rpy="${-90*M_PI/180} ${0*M_PI/180} ${-90*M_PI/180}"/> -->
             <parent
-                link="${image_link}"/>
+                link="${camera_link}"/>
             <child
                 link="${point_link}"/>
         </joint>
         <gazebo reference="${image_link}">
-            <sensor name="${object_name}_depth_sensor" type="depth">
+            <sensor
+                name="${object_name}_sensor"
+                type="rgbd_camera">
+                <!-- Sensor pose relative to image_link -->
+                <pose>0 0 0 0 0 0</pose>
                 <always_on>true</always_on>
                 <update_rate>30</update_rate>
                 <visualize>true</visualize>
-                <camera>
-                    <horizontal_fov>${60*M_PI/180}</horizontal_fov>
+                <!--
+                    Base Gazebo Transport topic.
+                    Expected child topics:
+                        ${topic}/image
+                        ${topic}/camera_info
+                        ${topic}/depth_image
+                        ${topic}/points
+                -->
+                <topic>${topic}</topic>
+                <!-- Gazebo rendering sensor frame: +Z forward -->
+                <gz_frame_id>${point_link}</gz_frame_id>
+                <camera name="${object_name}_camera">
+                    <horizontal_fov>
+                        ${60.0 * M_PI / 180.0}
+                    </horizontal_fov>
                     <image>
                         <width>640</width>
@@ -95,21 +126,21 @@
                         <format>R8G8B8</format>
                     </image>
+                    <!-- RGB rendering range -->
                     <clip>
                         <near>0.1</near>
                         <far>8.0</far>
                     </clip>
+                    <!-- Depth and point-cloud range -->
+                    <depth_camera>
+                        <clip>
+                            <near>0.2</near>
+                            <far>8.0</far>
+                        </clip>
+                    </depth_camera>
+                    <!-- ROS optical convention -->
+                    <optical_frame_id>
+                        ${image_link}
+                    </optical_frame_id>
                 </camera>
-                <plugin name="${object_name}_plugin" filename="libgazebo_ros_camera.so">
-                    <ros>
-                        <namespace>/</namespace>
-                        <remapping>${object_name}_depth_sensor/camera_info:=${topic}/camera_info</remapping>
-                        <remapping>${object_name}_depth_sensor/depth/camera_info:=${topic}/depth/camera_info</remapping>
-                        <remapping>${object_name}_depth_sensor/image_raw:=${topic}/image_raw</remapping>
-                        <remapping>${object_name}_depth_sensor/depth/image_raw:=${topic}/depth/image_raw</remapping>
-                        <remapping>${object_name}_depth_sensor/points:=${topic}/points</remapping>
-                    </ros>
-                    <frame_name>${point_link}</frame_name>
-                    <point_cloud_cutoff>0.2</point_cloud_cutoff>
-                </plugin>
             </sensor>
         </gazebo>

File: limo_bringup/description/urdf/limo_base.xacro (robot description, xacro)
@@ -1,5 +1,5 @@
 <?xml version="1.0"?>
-<robot name="base" xmlns:xacro="http://wiki.ros.org/xacro">
-    <xacro:macro name="base" params="object_name:='base' frame_link='base_link' parent_link:='base_footprint' xyz:='0 0 0' rpy:='0 0 0' color:='false' simple:='true'">
+<robot name="limo_base" xmlns:xacro="http://wiki.ros.org/xacro">
+    <xacro:macro name="limo_base" params="object_name:='limo_base' frame_link='base_link' parent_link:='base_footprint' xyz:='0 0 0' rpy:='0 0 0' color:='false' simple:='true'">
         <xacro:property
             name="mass"
@@ -41,10 +41,10 @@
                     <xacro:if value="${color}">
                         <mesh
-                            filename="file://$(find limo_description)/meshes/limo_base.dae"
+                            filename="file://$(find limo_bringup)/description/meshes/limo_base.dae"
                             scale="1 1 1"/>
                     </xacro:if>
                     <xacro:unless value="${color}">
                         <mesh
-                            filename="file://$(find limo_description)/meshes/limo_base.stl"
+                            filename="file://$(find limo_bringup)/description/meshes/limo_base.stl"
                             scale="0.001 0.001 0.001"/>
                     </xacro:unless>
@@ -76,10 +76,10 @@
                         <xacro:if value="${color}">
                             <mesh
-                                filename="file://$(find limo_description)/meshes/limo_base.dae"
+                                filename="file://$(find limo_bringup)/meshes/limo_base.dae"
                                 scale="1 1 1"/>
                         </xacro:if>
                         <xacro:unless value="${color}">
                             <mesh
-                                filename="file://$(find limo_description)/meshes/base_link.stl"
+                                filename="file://$(find limo_bringup)/meshes/base_link.stl"
                                 scale="0.001 0.001 0.001"/>
                         </xacro:unless>
@@ -100,11 +100,25 @@
         </joint>
         <gazebo reference="${frame_link}">
+            <!-- Link-level setting -->
             <gravity>true</gravity>
-            <kp>1000000.0</kp>
-            <kd>1.0</kd>
-            <mu1>0.8</mu1>
-            <mu2>0.8</mu2>
-            <maxVel>0.0</maxVel>
-            <minDepth>0.001</minDepth>
+            <!-- Inserted into the link collision -->
+            <collision>
+                <surface>
+                    <friction>
+                        <ode>
+                            <mu>0.8</mu>
+                            <mu2>0.8</mu2>
+                        </ode>
+                    </friction>
+                    <contact>
+                        <ode>
+                            <kp>1000000.0</kp>
+                            <kd>1.0</kd>
+                            <max_vel>0.0</max_vel>
+                            <min_depth>0.001</min_depth>
+                        </ode>
+                    </contact>
+                </surface>
+            </collision>
         </gazebo>
     </xacro:macro>

File: limo_bringup/description/urdf/limo_wheel.xacro (robot description, xacro)
@@ -1,5 +1,5 @@
 <?xml version="1.0"?>
-<robot name="wheel" xmlns:xacro="http://wiki.ros.org/xacro">
-    <xacro:macro name="wheel" params="object_name:='wheel' joint_name='wheel_joint' frame_link='wheel_link' parent_link:='base_link' xyz:='0 0 0' rpy:='0 0 0' direction:='1' color:='false' simple:='true'">
+<robot name="limo_wheel" xmlns:xacro="http://wiki.ros.org/xacro">
+    <xacro:macro name="limo_wheel" params="object_name:='limo_wheel' joint_name='limo_wheel_joint' frame_link='limo_wheel_link' parent_link:='base_link' xyz:='0 0 0' rpy:='0 0 0' direction:='1' color:='false' simple:='true'">
         <xacro:property
             name="mass"
@@ -37,10 +37,10 @@
                     <xacro:if value="${color}">
                         <mesh
-                            filename="file://$(find limo_description)/meshes/limo_wheel.dae"
+                            filename="file://$(find limo_bringup)/description/meshes/limo_wheel.dae"
                             scale="1 1 1"/>
                     </xacro:if>
                     <xacro:unless value="${color}">
                         <mesh
-                            filename="file://$(find limo_description)/meshes/limo_wheel.stl"
+                            filename="file://$(find limo_bringup)/description/meshes/limo_wheel.stl"
                             scale="0.001 0.001 0.001"/>
                     </xacro:unless>
@@ -72,10 +72,10 @@
                         <xacro:if value="${color}">
                             <mesh
-                                filename="file://$(find limo_description)/meshes/limo_wheel.dae"
+                                filename="file://$(find limo_bringup)/description/meshes/limo_wheel.dae"
                                 scale="1 1 1"/>
                         </xacro:if>
                         <xacro:unless value="${color}">
                             <mesh
-                                filename="file://$(find limo_description)/meshes/limo_wheel.stl"
+                                filename="file://$(find limo_bringup)/description/meshes/limo_wheel.stl"
                                 scale="0.001 0.001 0.001"/>
                         </xacro:unless>
@@ -97,5 +97,6 @@
                 xyz="0 ${direction} 0"/>
         </joint>
-        <transmission
+        <!-- this is for ros1 -->
+        <!-- <transmission
             name="${object_name}_trans"
             type="SimpleTransmission">
@@ -115,12 +116,34 @@
                 </mechanicalReduction>
             </actuator>
-        </transmission>
+        </transmission> -->
         <gazebo reference="${frame_link}">
-            <material>Gazebo/Black</material>
-            <kp>1000000.0</kp>
-            <kd>1.0</kd>
-            <mu1>1.0</mu1>
-            <mu2>0.5</mu2>
-            <fdir1>1 0 0</fdir1>
+            <!-- Link-level setting -->
+            <gravity>true</gravity>
+            <!-- Applied to every visual in this URDF link -->
+            <visual>
+                <material>
+                    <ambient>0.0 0.0 0.0 1.0</ambient>
+                    <diffuse>0.0 0.0 0.0 1.0</diffuse>
+                    <specular>0.0 0.0 0.0 1.0</specular>
+                </material>
+            </visual>
+            <!-- Applied to every collision in this URDF link -->
+            <collision>
+                <surface>
+                    <friction>
+                        <ode>
+                            <mu>1.0</mu>
+                            <mu2>0.5</mu2>
+                            <fdir1>1 0 0</fdir1>
+                        </ode>
+                    </friction>
+                    <contact>
+                        <ode>
+                            <kp>1000000.0</kp>
+                            <kd>1.0</kd>
+                        </ode>
+                    </contact>
+                </surface>
+            </collision>
         </gazebo>
     </xacro:macro>

File: limo_bringup/description/urdf/ydlidar.xacro (robot description, xacro)
@@ -70,14 +70,17 @@
         </joint>
         <gazebo reference="${frame_link}">
-            <sensor name="${object_name}" type="ray">
+            <sensor name="${object_name}_sensor" type="gpu_lidar">
                 <pose>0 0 0 0 0 0</pose>
+                <always_on>true</always_on>
                 <visualize>true</visualize>
                 <update_rate>10</update_rate>
-                <ray>
+                <topic>${topic}</topic>
+                <gz_frame_id>${frame_link}</gz_frame_id>
+                <lidar>
                     <scan>
                         <horizontal>
                             <samples>461</samples>
                             <resolution>1</resolution>
-                            <min_angle>-${M_PI}</min_angle>
+                            <min_angle>${-M_PI}</min_angle>
                             <max_angle>${M_PI}</max_angle>
                         </horizontal>
@@ -93,14 +96,5 @@
                         <stddev>0.01</stddev>
                     </noise>
-                </ray>
-                <plugin name="${object_name}_plugin" filename="libgazebo_ros_ray_sensor.so">
-                    <ros>
-                        <namespace>/</namespace>
-                        <remapping>${object_name}_plugin/out:=${topic}</remapping>
-                    </ros>
-                    <output_type>sensor_msgs/LaserScan</output_type>
-                    <frame_name>${frame_link}</frame_name>
-                    <gaussian_noise>0.01</gaussian_noise>
-                </plugin>
+                </lidar>
             </sensor>
         </gazebo>
